Commit message: fixed wrong format for number

File: robot_model/mpo_700/xacros/sick_s300_laser.xacro (robot description, xacro)
@@ -15,5 +15,5 @@
       </inertial>
       <visual>
-        <origin xyz="0 0 0.0" rpy="0 0 -1,57" />
+        <origin xyz="0 0 0.0" rpy="0 0 -1.57" />
         <geometry>
           <mesh filename="package://neo_mpo_700/robot_model/mpo_700/meshes/MPO-700-SICK.STL" />
