Commit message: fixed robot model

File: robot_model/mpo_700/mpo_700.urdf.xacro (robot description, xacro)
@@ -2,10 +2,10 @@
 <robot name="mpo_700" xmlns:xacro="http://www.ros.org/wiki/xacro">
   <!-- MATERIALS -->
-  <xacro:include filename="$(find neo_simulation)/robots/mpo_700/xacros/mpo_700_materials.xacro" />
+  <xacro:include filename="$(find neo_mpo_700)/robot_model/mpo_700/xacros/mpo_700_materials.xacro" />
   <!-- BODY -->
-  <xacro:include filename="$(find neo_simulation)/robots/mpo_700/xacros/mpo_700_body.xacro" />
+  <xacro:include filename="$(find neo_mpo_700)/robot_model/mpo_700/xacros/mpo_700_body.xacro" />
   <!-- SENSORS -->
-  <xacro:include filename="$(find neo_simulation)/robots/mpo_700/xacros/sick_s300_laser.xacro" />
-  <xacro:include filename="$(find neo_simulation)/robots/mpo_700/xacros/mpo_700_gazebo.xacro" />
+  <xacro:include filename="$(find neo_mpo_700)/robot_model/mpo_700/xacros/sick_s300_laser.xacro" />
+  <xacro:include filename="$(find neo_mpo_700)/robot_model/mpo_700/xacros/mpo_700_gazebo.xacro" />
   <!-- Base Macro-->
   <xacro:mpo_700_base name="base_link">

File: robot_model/mpo_700/xacros/mpo_700_body.xacro (robot description, xacro)
@@ -13,5 +13,5 @@
         <origin xyz="0.0 0.0 0.021" rpy="0 0 1.571" />
         <geometry>
-            <mesh filename="package://neo_simulation/robots/mpo_700/meshes/MPO-700.stl" scale="0.001 0.001 0.001"/>
+            <mesh filename="package://neo_mpo_700/robot_model/mpo_700/meshes/MPO-700.stl" scale="0.001 0.001 0.001"/>
         </geometry>
         <material name="Neobotix/Grey" />

File: robot_model/mpo_700/xacros/sick_s300_laser.xacro (robot description, xacro)
@@ -17,5 +17,5 @@
         <origin xyz="0 0 0.0" rpy="0 0 0" />
         <geometry>
-          <mesh filename="package://neo_simulation/robots/mpo_700/meshes/MPO-700-SICK.STL" />
+          <mesh filename="package://neo_mpo_700/robot_model/mpo_700/meshes/MPO-700-SICK.STL" />
         </geometry>
         <material name="Neobotix/Yellow" />

Commit message: fixed hardware parameter, fixed robot model scanner positions, fixed EM-Stop topic names, added auto_recover

File: robot_model/mpo_700/mpo_700.urdf.xacro (robot description, xacro)
@@ -13,8 +13,8 @@
   <!-- Sensors -->
   <xacro:sick_s300_laser_v0 name="sick_s300_laser_front" parent="base_link" ros_topic="sick_s300_front/scan">
-  	<origin xyz="0.360 0 0.223" rpy="3.14 0 1.57" />
+  	<origin xyz="0.360 0 0.223" rpy="3.14 0 0" />
   </xacro:sick_s300_laser_v0>
   <xacro:sick_s300_laser_v0 name="sick_s300_laser_back" parent="base_link" ros_topic="sick_s300_back/scan">
-  	<origin xyz="-0.360 0 0.223" rpy="3.14 0 -1.57" />
+  	<origin xyz="-0.360 0 0.223" rpy="3.14 0 -3.14" />
   </xacro:sick_s300_laser_v0>
 </robot>

File: robot_model/mpo_700/xacros/sick_s300_laser.xacro (robot description, xacro)
@@ -15,5 +15,5 @@
       </inertial>
       <visual>
-        <origin xyz="0 0 0.0" rpy="0 0 0" />
+        <origin xyz="0 0 0.0" rpy="0 0 -1,57" />
         <geometry>
           <mesh filename="package://neo_mpo_700/robot_model/mpo_700/meshes/MPO-700-SICK.STL" />

Commit message: updated robot model and added .launch file for visualization

File: robot_model/mpo_700/mpo_700.urdf.xacro (robot description, xacro)
@@ -1,20 +1,43 @@
 <?xml version="1.0" ?>
 <robot name="mpo_700" xmlns:xacro="http://www.ros.org/wiki/xacro">
-  <!-- MATERIALS -->
-  <xacro:include filename="$(find neo_mpo_700)/robot_model/mpo_700/xacros/mpo_700_materials.xacro" />
   <!-- BODY -->
   <xacro:include filename="$(find neo_mpo_700)/robot_model/mpo_700/xacros/mpo_700_body.xacro" />
   <!-- SENSORS -->
-  <xacro:include filename="$(find neo_mpo_700)/robot_model/mpo_700/xacros/sick_s300_laser.xacro" />
-  <!--xacro:include filename="$(find neo_mpo_700)/robot_model/mpo_700/xacros/mpo_700_gazebo.xacro" /-->
+  <xacro:include filename="$(find neo_mpo_700)/robot_model/mpo_700/xacros/sick_laser.xacro" />
+  <xacro:include filename="$(find neo_mpo_700)/robot_model/mpo_700/xacros/mpo_700_head.xacro" />
+  <xacro:include filename="$(find neo_mpo_700)/robot_model/mpo_700/xacros/mpo_700_wheel.xacro" />
   <!-- Base Macro-->
   <xacro:mpo_700_base name="base_link">
   </xacro:mpo_700_base>
-  <!-- Sensors -->
-  <xacro:sick_s300_laser_v0 name="sick_s300_laser_front" parent="base_link" ros_topic="sick_s300_front/scan">
-  	<origin xyz="0.360 0 0.223" rpy="3.14 0 0" />
-  </xacro:sick_s300_laser_v0>
-  <xacro:sick_s300_laser_v0 name="sick_s300_laser_back" parent="base_link" ros_topic="sick_s300_back/scan">
-  	<origin xyz="-0.360 0 0.223" rpy="3.14 0 -3.14" />
-  </xacro:sick_s300_laser_v0>
+<xacro:mpo_700_head_0 name="mpo_700_head_0" parent="base_link">
+    <origin xyz="0.24 0.18 0.27" rpy="3.14 0 -1.57" />
+  </xacro:mpo_700_head_0>
+<xacro:mpo_700_head_1 name="mpo_700_head_1" parent="base_link">
+    <origin xyz="0.24 -0.18 0.27" rpy="3.14 0 1.57" />
+  </xacro:mpo_700_head_1>
+<xacro:mpo_700_head_2 name="mpo_700_head_2" parent="base_link">
+    <origin xyz="-0.24 0.18 0.27" rpy="3.14 0 -1.57" />
+  </xacro:mpo_700_head_2>
+<xacro:mpo_700_head_3 name="mpo_700_head_3" parent="base_link">
+    <origin xyz="-0.24 -0.18 0.27" rpy="3.14 0 1.57" />
+  </xacro:mpo_700_head_3>
+<xacro:mpo_700_wheel name="wheel_0" parent="mpo_700_head_0_link">
+    <origin xyz="-0.05 0. 0.18" rpy="0 0 0" />
+  </xacro:mpo_700_wheel>
+<xacro:mpo_700_wheel name="wheel_1" parent="mpo_700_head_1_link">
+    <origin xyz="-0.05 0. 0.18" rpy="0 0 0" />
+  </xacro:mpo_700_wheel>
+<xacro:mpo_700_wheel name="wheel_2" parent="mpo_700_head_2_link">
+    <origin xyz="-0.05 0. 0.18" rpy="0 0 0" />
+  </xacro:mpo_700_wheel>
+<xacro:mpo_700_wheel name="wheel_3" parent="mpo_700_head_3_link">
+    <origin xyz="-0.05 0. 0.18" rpy="0 0 0" />
+  </xacro:mpo_700_wheel>
+<!-- Sensors -->
+  <xacro:sick_v0 name="laser_1" parent="base_link" ros_topic="sick_front/scan">
+  	<origin xyz="0.360 0 0.181" rpy="3.14 0 0 " />
+  </xacro:sick_v0>
+  <xacro:sick_v0 name="laser_2" parent="base_link" ros_topic="sick_back/scan">
+  	<origin xyz="-0.360 0 0.181" rpy="3.14 0 3.14" />
+  </xacro:sick_v0>
 </robot>

File: robot_model/mpo_700/xacros/mpo_700_body.xacro (robot description, xacro)
@@ -11,14 +11,13 @@
       </inertial>
       <visual>
-        <origin xyz="0.0 0.0 0.021" rpy="0 0 1.571" />
+        <origin xyz="0.0 0.0 0.0" rpy="0 0 -1.571" />
         <geometry>
-            <mesh filename="package://neo_mpo_700/robot_model/mpo_700/meshes/MPO-700.stl" scale="0.001 0.001 0.001"/>
+            <mesh filename="package://neo_mpo_700/robot_model/mpo_700/meshes/MPO-700-BODY.dae" scale="0.001 0.001 0.001"/>
         </geometry>
-        <material name="Neobotix/Grey" />
       </visual>
       <collision>
-        <origin xyz="0. 0. 0.2" rpy="0 0 0" />
+        <origin xyz="0. 0. 0." rpy="0 0 -1.571" />
         <geometry>
-          <box size="0.610 0.515 0.360" />
+            <mesh filename="package://neo_mpo_700/robot_model/mpo_700/meshes/MPO-700-BODY.dae" scale="0.001 0.001 0.001"/>
         </geometry>
       </collision>

Commit message: added laser positions for both options

File: robot_model/mpo_700/mpo_700.urdf.xacro (robot description, xacro)
@@ -36,8 +36,10 @@
 <!-- Sensors -->
   <xacro:sick_v0 name="laser_1" parent="base_link" ros_topic="sick_front/scan">
-  	<origin xyz="0.360 0 0.181" rpy="3.14 0 0 " />
+	<!--<origin xyz="0.360 0 0.181" rpy="3.14 0 0" />-->
+  	<origin xyz="0.338 0.288 0.223" rpy="3.14 0 0.79" />
   </xacro:sick_v0>
   <xacro:sick_v0 name="laser_2" parent="base_link" ros_topic="sick_back/scan">
-  	<origin xyz="-0.360 0 0.181" rpy="3.14 0 3.14" />
+	<!--<origin xyz="-0.360 0 0.181" rpy="3.14 0 3.14" />-->
+  	<origin xyz="-0.338 -0.288 0.223" rpy="3.14 0 3.93" />
   </xacro:sick_v0>
 </robot>

Commit message: added frames for IMU and USSensors to robot model

File: robot_model/mpo_700/mpo_700.urdf.xacro (robot description, xacro)
@@ -43,3 +43,75 @@
   	<origin xyz="-0.338 -0.288 0.223" rpy="3.14 0 3.93" />
   </xacro:sick_v0>
+  <!--+++++++++++++++++++ IMU ++++++++++++++++++++++++-->
+  <!-- SENSORS -->
+  <xacro:include filename="$(find neo_mpo_700)/robot_model/mpo_700/xacros/imu.xacro" />
+  <xacro:imu name="imu_1" parent="base_link">
+    <origin xyz="0.100 0 0.300" rpy="0 0 3.14" />
+  </xacro:imu>
+  <!--+++++++++++++++++++ Ultra Sonic ++++++++++++++++++++++++-->
+  <xacro:include filename="$(find neo_mpo_700)/robot_model/mpo_700/xacros/ultrasonic.xacro" />
+  <!-- SENSOR 1 -->
+  <!-- xacro:us_sensor name="us_1" parent="base_link">
+    <origin xyz="0.100 0 0.300" rpy="0 3.14 3.14" />
+  </xacro:us_sensor-->
+  <!-- SENSOR 2 -->
+  <!-- xacro:us_sensor name="us_2" parent="base_link">
+    <origin xyz="0.110 0 0.300" rpy="0 3.14 3.14" />
+  </xacro:us_sensor-->
+  <!-- SENSOR 3 -->
+  <!-- xacro:us_sensor name="us_3" parent="base_link">
+    <origin xyz="0.120 0 0.300" rpy="0 3.14 3.14" />
+  </xacro:us_sensor-->
+  <!-- SENSOR 4 -->
+  <!-- xacro:us_sensor name="us_4" parent="base_link">
+    <origin xyz="0.130 0 0.300" rpy="0 3.14 3.14" />
+  </xacro:us_sensor-->
+  <!-- SENSOR 5 -->
+  <!-- xacro:us_sensor name="us_5" parent="base_link">
+    <origin xyz="0.140 0 0.300" rpy="0 3.14 3.14" />
+  </xacro:us_sensor-->
+  <!-- SENSOR 6 -->
+  <!-- xacro:us_sensor name="us_6" parent="base_link">
+    <origin xyz="0.150 0 0.300" rpy="0 3.14 3.14" />
+  </xacro:us_sensor-->
+  <!-- SENSOR 7 -->
+  <!-- xacro:us_sensor name="us_7" parent="base_link">
+    <origin xyz="0.160 0 0.300" rpy="0 3.14 3.14" />
+  </xacro:us_sensor-->
+  <!-- SENSOR 8 -->
+  <!-- xacro:us_sensor name="us_8" parent="base_link">
+    <origin xyz="0.170 0 0.300" rpy="0 3.14 3.14" />
+  </xacro:us_sensor-->
+  <!-- SENSOR 9 -->
+  <!-- xacro:us_sensor name="us_9" parent="base_link">
+    <origin xyz="0.180 0 0.300" rpy="0 3.14 3.14" />
+  </xacro:us_sensor-->
+  <!-- SENSOR 10 -->
+  <!-- xacro:us_sensor name="us_10" parent="base_link">
+    <origin xyz="0.100 0 0.300" rpy="0 3.14 3.14" />
+  </xacro:us_sensor-->
+  <!-- SENSOR 11 -->
+  <!-- xacro:us_sensor name="us_11" parent="base_link">
+    <origin xyz="0.100 0 0.300" rpy="0 3.14 3.14" />
+  </xacro:us_sensor-->
+  <!-- SENSOR 12 -->
+  <!-- xacro:us_sensor name="us_12" parent="base_link">
+    <origin xyz="0.190 0 0.300" rpy="0 3.14 3.14" />
+  </xacro:us_sensor-->
+  <!-- SENSOR 13 -->
+  <!-- xacro:us_sensor name="us_13" parent="base_link">
+    <origin xyz="0.200 0 0.300" rpy="0 3.14 3.14" />
+  </xacro:us_sensor-->
+  <!-- SENSOR 14 -->
+  <!-- xacro:us_sensor name="us_14" parent="base_link">
+    <origin xyz="0.210 0 0.300" rpy="0 3.14 3.14" />
+  </xacro:us_sensor-->
+  <!-- SENSOR 15 -->
+  <!-- xacro:us_sensor name="us_15" parent="base_link">
+    <origin xyz="0.220 0 0.300" rpy="0 3.14 3.14" />
+  </xacro:us_sensor-->
+  <!-- SENSOR 16 -->
+  <!-- xacro:us_sensor name="us_16" parent="base_link">
+    <origin xyz="0.230 0 0.300" rpy="0 3.14 3.14" />
+  </xacro:us_sensor-->
 </robot>

Commit message: Added sensors

File: robot_model/mpo_700/mpo_700.urdf.xacro (robot description, xacro)
@@ -4,5 +4,11 @@
   <xacro:include filename="$(find neo_mpo_700)/robot_model/mpo_700/xacros/mpo_700_body.xacro" />
   <!-- SENSORS -->
-  <xacro:include filename="$(find neo_mpo_700)/robot_model/mpo_700/xacros/sick_laser.xacro" />
+  <!-- Sick S300 - Comment/Uncomment if required -->
+  <xacro:include filename="$(find neo_mpo_700)/robot_model/mpo_700/xacros/sick_S300.xacro" />
+  <!-- Microscan - Comment/Uncomment if required -->
+  <!-- <xacro:include filename="$(find neo_mpo_700)/robot_model/mpo_700/xacros/micro_scan.xacro" />  -->
+  <!--<xacro:include filename="$(find neo_mpo_700)/robot_model/mpo_700/xacros/imu.xacro" />
+  <xacro:include filename="$(find neo_mpo_700)/robot_model/mpo_700/xacros/ultrasonic.xacro" /> -->
+  <xacro:include filename="$(find neo_mpo_700)/robot_model/mpo_700/xacros/mpo_700_gazebo.xacro" />
   <xacro:include filename="$(find neo_mpo_700)/robot_model/mpo_700/xacros/mpo_700_head.xacro" />
   <xacro:include filename="$(find neo_mpo_700)/robot_model/mpo_700/xacros/mpo_700_wheel.xacro" />
@@ -35,11 +41,85 @@
   </xacro:mpo_700_wheel>
 <!-- Sensors -->
-  <xacro:sick_v0 name="lidar_1" parent="base_link" ros_topic="sick_front/scan">
-	<!--<origin xyz="0.360 0 0.181" rpy="3.14 0 0" />-->
-  	<origin xyz="0.338 0.288 0.223" rpy="3.14 0 0.79" />
-  </xacro:sick_v0>
-  <xacro:sick_v0 name="lidar_2" parent="base_link" ros_topic="sick_back/scan">
-	<!--<origin xyz="-0.360 0 0.181" rpy="3.14 0 3.14" />-->
-  	<origin xyz="-0.338 -0.288 0.223" rpy="3.14 0 3.93" />
-  </xacro:sick_v0>
+  <xacro:sick_laser_v0 name="lidar_1" parent="base_link" ros_topic="lidar_1/scan_filtered">
+  	<origin xyz="0.360 0 0.181" rpy="3.14 0 0 " />
+  </xacro:sick_laser_v0>
+  <xacro:sick_laser_v0 name="lidar_2" parent="base_link" ros_topic="lidar_2/scan_filtered">
+  	<origin xyz="-0.360 0 0.181" rpy="3.14 0 3.14" />
+  </xacro:sick_laser_v0>
+     <!--+++++++++++++++++++ IMU ++++++++++++++++++++++++-->
+ <!-- Comment or uncomment based on your requirement -->
+<!--   <xacro:imu name="imu_1" parent="base_link">
+    <origin xyz="0.100 0 0.300" rpy="0 0 3.14" />
+  </xacro:imu> -->
+  <!--+++++++++++++++++++ Ultra Sonic ++++++++++++++++++++++++-->
+  <!-- Comment or uncomment based on your requirement -->
+  <!-- SENSOR 1 -->
+  <!-- xacro:us_sensor name="us_1" parent="base_link">
+    <origin xyz="0.100 0 0.300" rpy="0 3.14 3.14" />
+  </xacro:us_sensor-->
+  <!-- SENSOR 2 -->
+  <!-- xacro:us_sensor name="us_2" parent="base_link">
+    <origin xyz="0.110 0 0.300" rpy="0 3.14 3.14" />
+  </xacro:us_sensor-->
+  <!-- SENSOR 3 -->
+  <!-- xacro:us_sensor name="us_3" parent="base_link">
+    <origin xyz="0.120 0 0.300" rpy="0 3.14 3.14" />
+  </xacro:us_sensor-->
+  <!-- SENSOR 4 -->
+  <!-- xacro:us_sensor name="us_4" parent="base_link">
+    <origin xyz="0.130 0 0.300" rpy="0 3.14 3.14" />
+  </xacro:us_sensor-->
+  <!-- SENSOR 5 -->
+  <!-- xacro:us_sensor name="us_5" parent="base_link">
+    <origin xyz="0.140 0 0.300" rpy="0 3.14 3.14" />
+  </xacro:us_sensor-->
+  <!-- SENSOR 6 -->
+  <!-- xacro:us_sensor name="us_6" parent="base_link">
+    <origin xyz="0.150 0 0.300" rpy="0 3.14 3.14" />
+  </xacro:us_sensor-->
+  <!-- SENSOR 7 -->
+  <!-- xacro:us_sensor name="us_7" parent="base_link">
+    <origin xyz="0.160 0 0.300" rpy="0 3.14 3.14" />
+  </xacro:us_sensor-->
+  <!-- SENSOR 8 -->
+  <!-- xacro:us_sensor name="us_8" parent="base_link">
+    <origin xyz="0.170 0 0.300" rpy="0 3.14 3.14" />
+  </xacro:us_sensor-->
+  <!-- SENSOR 9 -->
+  <!-- xacro:us_sensor name="us_9" parent="base_link">
+    <origin xyz="0.180 0 0.300" rpy="0 3.14 3.14" />
+  </xacro:us_sensor-->
+  <!-- SENSOR 10 -->
+  <!-- xacro:us_sensor name="us_10" parent="base_link">
+    <origin xyz="0.100 0 0.300" rpy="0 3.14 3.14" />
+  </xacro:us_sensor-->
+  <!-- SENSOR 11 -->
+  <!-- xacro:us_sensor name="us_11" parent="base_link">
+    <origin xyz="0.100 0 0.300" rpy="0 3.14 3.14" />
+  </xacro:us_sensor-->
+  <!-- SENSOR 12 -->
+  <!-- xacro:us_sensor name="us_12" parent="base_link">
+    <origin xyz="0.190 0 0.300" rpy="0 3.14 3.14" />
+  </xacro:us_sensor-->
+  <!-- SENSOR 13 -->
+  <!-- xacro:us_sensor name="us_13" parent="base_link">
+    <origin xyz="0.200 0 0.300" rpy="0 3.14 3.14" />
+  </xacro:us_sensor-->
+  <!-- SENSOR 14 -->
+  <!-- xacro:us_sensor name="us_14" parent="base_link">
+    <origin xyz="0.210 0 0.300" rpy="0 3.14 3.14" />
+  </xacro:us_sensor-->
+  <!-- SENSOR 15 -->
+  <!-- xacro:us_sensor name="us_15" parent="base_link">
+    <origin xyz="0.220 0 0.300" rpy="0 3.14 3.14" />
+  </xacro:us_sensor-->
+  <!-- SENSOR 16 -->
+  <!-- xacro:us_sensor name="us_16" parent="base_link">
+    <origin xyz="0.230 0 0.300" rpy="0 3.14 3.14" />
+  </xacro:us_sensor-->
+      <!--Camera  -->
+<!-- <xacro:camera name="camera" parent="base_link">
+    <origin xyz="0 0 0.38" rpy="0 0 0" />
+  </xacro:camera>
+ -->
 </robot>

Commit message: Laser positions updated

File: robot_model/mpo_700/mpo_700.urdf.xacro (robot description, xacro)
@@ -42,8 +42,10 @@
 <!-- Sensors -->
   <xacro:sick_laser_v0 name="lidar_1" parent="base_link" ros_topic="lidar_1/scan_filtered">
-  	<origin xyz="0.360 0 0.181" rpy="3.14 0 0 " />
+    <origin xyz="0.360 0 0.181" rpy="3.14 0 0" /> <!-- Scanners on the side -->
+  	<!-- <origin xyz="0.360 0 0.181" rpy="3.14 0 0 " /> --> <!-- Scanners on the front -->
   </xacro:sick_laser_v0>
   <xacro:sick_laser_v0 name="lidar_2" parent="base_link" ros_topic="lidar_2/scan_filtered">
-  	<origin xyz="-0.360 0 0.181" rpy="3.14 0 3.14" />
+    <origin xyz="-0.360 0 0.181" rpy="3.14 0 3.14" /> <!-- Scanners on the side -->
+  	<!-- <origin xyz="-0.360 0 0.181" rpy="3.14 0 3.14" /> --> <!-- Scanners on the bsck -->
   </xacro:sick_laser_v0>
      <!--+++++++++++++++++++ IMU ++++++++++++++++++++++++-->

Commit message: Scanners are added on the corner

File: robot_model/mpo_700/mpo_700.urdf.xacro (robot description, xacro)
@@ -42,10 +42,10 @@
 <!-- Sensors -->
   <xacro:sick_laser_v0 name="lidar_1" parent="base_link" ros_topic="lidar_1/scan_filtered">
-    <origin xyz="0.360 0 0.181" rpy="3.14 0 0" /> <!-- Scanners on the side -->
-  	<!-- <origin xyz="0.360 0 0.181" rpy="3.14 0 0 " /> --> <!-- Scanners on the front -->
+  <!--<origin xyz="0.360 0 0.181" rpy="3.14 0 0" />-->
+    <origin xyz="0.338 0.288 0.223" rpy="3.14 0 0.79" /> <!-- Scanners on the side -->
   </xacro:sick_laser_v0>
   <xacro:sick_laser_v0 name="lidar_2" parent="base_link" ros_topic="lidar_2/scan_filtered">
-    <origin xyz="-0.360 0 0.181" rpy="3.14 0 3.14" /> <!-- Scanners on the side -->
-  	<!-- <origin xyz="-0.360 0 0.181" rpy="3.14 0 3.14" /> --> <!-- Scanners on the bsck -->
+  <!--<origin xyz="-0.360 0 0.181" rpy="3.14 0 3.14" />-->
+    <origin xyz="-0.338 -0.288 0.223" rpy="3.14 0 3.93" /> <!-- Scanners on the side -->
   </xacro:sick_laser_v0>
      <!--+++++++++++++++++++ IMU ++++++++++++++++++++++++-->

Commit message: Visualization of camera model added.

File: robot_model/mpo_700/mpo_700.urdf.xacro (robot description, xacro)
@@ -10,4 +10,6 @@
   <!--<xacro:include filename="$(find neo_mpo_700)/robot_model/mpo_700/xacros/imu.xacro" />
   <xacro:include filename="$(find neo_mpo_700)/robot_model/mpo_700/xacros/ultrasonic.xacro" /> -->
+  <!-- Depth Camera -->
+  <xacro:include filename="$(find neo_mpo_700)/robot_model/mpo_700/xacros/depth_camera.xacro" />
   <xacro:include filename="$(find neo_mpo_700)/robot_model/mpo_700/xacros/mpo_700_gazebo.xacro" />
   <xacro:include filename="$(find neo_mpo_700)/robot_model/mpo_700/xacros/mpo_700_head.xacro" />
@@ -120,8 +122,11 @@
     <origin xyz="0.230 0 0.300" rpy="0 3.14 3.14" />
   </xacro:us_sensor-->
-      <!--Camera  -->
-<!-- <xacro:camera name="camera" parent="base_link">
+  <!-- Camera -->
+  <!-- xacro:camera name="camera" parent="base_link">
     <origin xyz="0 0 0.38" rpy="0 0 0" />
-  </xacro:camera>
- -->
+  </xacro:camera-->
+  <!-- Depth Camera -->
+  <!-- xacro:depth_camera name="camera" parent="base_link">
+    <origin xyz="0.228 0 0.461" rpy="0 0 0" />
+  </xacro:depth_camera-->
 </robot>

Commit message: Added dummy link and depreceated tags are removed

File: robot_model/mpo_700/mpo_700.urdf.xacro (robot description, xacro)
@@ -15,6 +15,8 @@
   <xacro:include filename="$(find neo_mpo_700)/robot_model/mpo_700/xacros/mpo_700_head.xacro" />
   <xacro:include filename="$(find neo_mpo_700)/robot_model/mpo_700/xacros/mpo_700_wheel.xacro" />
+  <link name="dummy_link" />
   <!-- Base Macro-->
-  <xacro:mpo_700_base name="base_link">
+  <xacro:mpo_700_base name="base_link" parent="dummy_link">
+    <origin xyz="0 0 0" rpy="0 0 0" />
   </xacro:mpo_700_base>
 <xacro:mpo_700_head_0 name="mpo_700_head_0" parent="base_link">

File: robot_model/mpo_700/xacros/mpo_700_body.xacro (robot description, xacro)
@@ -1,6 +1,14 @@
 <?xml version="1.0"?>
 <robot xmlns:xacro="http://www.ros.org/wiki/xacro" name="mpo_700">
-  <xacro:macro name="mpo_700_base" params="name">
-    <link name="${name}">
+  <xacro:macro name="mpo_700_base" params="name parent *origin">
+   <joint name="${name}_joint" type="fixed">
+    <insert_block name="origin" />
+    <axis xyz="0 0 -1" />
+    <!-- <limit effort="1000.0" lower="-1e+16" upper="1e+16" velocity="3.5"/> -->
+    <joint_properties damping="1" friction="1" />
+    <parent link="${parent}" />
+    <child link="${name}" />
+   </joint>
+   <link name="${name}">
       <inertial>
         <mass value="30" />

Commit message: URDF fix for rViz

File: robot_model/mpo_700/mpo_700.urdf.xacro (robot description, xacro)
@@ -15,19 +15,19 @@
   <xacro:include filename="$(find neo_mpo_700)/robot_model/mpo_700/xacros/mpo_700_head.xacro" />
   <xacro:include filename="$(find neo_mpo_700)/robot_model/mpo_700/xacros/mpo_700_wheel.xacro" />
-  <link name="dummy_link" />
+  <link name="base_link" />
   <!-- Base Macro-->
-  <xacro:mpo_700_base name="base_link" parent="dummy_link">
+  <xacro:mpo_700_base name="base_footprint" parent="base_link">
     <origin xyz="0 0 0" rpy="0 0 0" />
   </xacro:mpo_700_base>
-<xacro:mpo_700_head_0 name="mpo_700_head_0" parent="base_link">
+<xacro:mpo_700_head_0 name="mpo_700_head_0" parent="base_footprint">
     <origin xyz="0.24 0.18 0.27" rpy="3.14 0 -1.57" />
   </xacro:mpo_700_head_0>
-<xacro:mpo_700_head_1 name="mpo_700_head_1" parent="base_link">
+<xacro:mpo_700_head_1 name="mpo_700_head_1" parent="base_footprint">
     <origin xyz="0.24 -0.18 0.27" rpy="3.14 0 1.57" />
   </xacro:mpo_700_head_1>
-<xacro:mpo_700_head_2 name="mpo_700_head_2" parent="base_link">
+<xacro:mpo_700_head_2 name="mpo_700_head_2" parent="base_footprint">
     <origin xyz="-0.24 0.18 0.27" rpy="3.14 0 -1.57" />
   </xacro:mpo_700_head_2>
-<xacro:mpo_700_head_3 name="mpo_700_head_3" parent="base_link">
+<xacro:mpo_700_head_3 name="mpo_700_head_3" parent="base_footprint">
     <origin xyz="-0.24 -0.18 0.27" rpy="3.14 0 1.57" />
   </xacro:mpo_700_head_3>
